File: schematic/RaArPr/motherborard/motherborard.kicad_pcb (KiCad board)
At the start: 4 copper layers, 16 parts, among them J1 Conn_02x40_Odd_Even, SW1 SW_MEC_5E, U1 8088_Min_Mode, U2 74LS373, U3 8284, U4 74LS138, U5 74LS08, U6 74LS373, U7 74LS00, U8 AS6C4008-55PCN, U9 28C256, Y1 Crystal

Commit message: PCB
Routing:
- net A12: track 93.9 -> 217.7 mm, vias 0 -> 1
- net A8: track 121.2 -> 242.4 mm, vias 1 -> 2
- net AD6: track 157.5 -> 211.5 mm, vias 2 -> 3
- net +5V: track 313.4 -> 342.4 mm, vias 0 -> 1
- net GND: track 414.1 -> 422.8 mm
Other:
- board outline added: 116 x 111 mm
- board text added: "IGA CORP 80C88 CPU BOARD 512KB RAM 32KB ROM"
